Commit message: fix model

File: src/test_bot/description/robot_core.xacro (robot description, xacro)
@@ -56,5 +56,5 @@
         <parent link="base_link"/>
         <child link="left_wheel"/>
-        <origin xyz="0 0.113 0" rpy="-${pi/2} 0 0" />
+        <origin xyz="0 0.085 0" rpy="-${pi/2} 0 0" />
         <axis xyz="0 0 1"/>
         <!-- FIX: damping evita micro-movimientos espurios del simulador en reposo -->
@@ -93,5 +93,5 @@
         <parent link="base_link"/>
         <child link="right_wheel"/>
-        <origin xyz="0 -0.113 0" rpy="${pi/2} 0 0" />
+        <origin xyz="0 -0.085 0" rpy="${pi/2} 0 0" />
         <axis xyz="0 0 -1"/>
         <dynamics damping="0.05" friction="0.01"/>
